Commit message: modify the orientation of hips

File: robot.urdf (robot description, URDF)
Before this commit: robot dynamic_robot, 13 links, 12 joints
Joints:
- joint hipLB: origin xyz=0 0.062 0 rpy=1.57 0 0 -> xyz=0 0.062 0 rpy=-1.57 0 0
- joint hipLF: origin xyz=0 0.062 0 rpy=-1.57 0 0 -> xyz=0 0.062 0 rpy=1.57 0 0
- joint hipRB: origin xyz=0 0.062 0 rpy=-1.57 0 0 -> xyz=0 0.062 0 rpy=1.57 0 0
- joint hipRF: origin xyz=0 0.062 0 rpy=1.57 0 0 -> xyz=0 0.062 0 rpy=-1.57 0 0
